File: PowerSupply/PowerSupply.kicad_sch (KiCad schematic)
At the start: 15 parts, among them J1 POWER, J2 VSET, J3 LASER, U0 AL8861Y-13

Commit message: Resolve comments in second review
Parts:
- U0: footprint SOT89-5 -> Package_TO_SOT_SMD:SOT-89-5
Changed lines of the file:
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@@
     )
     (property "Value" "AL8861Y-13" (id 1) (at 171.45 95.25 0))
-    (property "Footprint" "SOT89-5" (id 2) (at 162.56 74.93 0)
+    (property "Footprint" "Package_TO_SOT_SMD:SOT-89-5" (id 2) (at 162.56 74.93 0)
       (effects (font (size 1.27 1.27)) (justify left bottom) hide)
     )
@@
     )
     (path "/31ddefd3-1a8e-42d5-a5b9-a7a71a2b2753"
-      (reference "U0") (unit 1) (value "AL8861Y-13") (footprint "SOT89-5")
-    )
-  )
+      (reference "U0") (unit 1) (value "AL8861Y-13") (footprint "Package_TO_SOT_SMD:SOT-89-5")
+    )
+  )
